File: kikad/toco_rev2/toco_rev2.kicad_sch (KiCad schematic)
At the start: 16 parts, among them M1 Motor_DC, Q1 NPN, SW1 SW_Push, SW10 SW_Push, SW11 SW_DPST_x2, SW2 SW_Push, SW3 SW_Push, SW4 SW_Push, SW5 SW_Push, SW6 SW_Push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

Commit message: fiddling whith pcb
Parts:
- removed D1: D, project:D3_TH_SMD_v2, symbol Device:D
- added D2: 1N4148W, Diode_SMD:D_SOD-123, symbol Diode:1N4148W
- BT1, M1: footprint (none) -> Connector_Wire:SolderWire-0.5sqmm_1x02_P4.6mm_D0.9mm_OD2.1mm
- SW11: footprint (none) -> Button_Switch_SMD:SW_SPDT_PCM12
Connections:
- net rumbler: now also U1.6 (A9_SCL/0.05_H); no longer U1.1 (A2/0.02_H)
- net switch01: now also U1.1 (A2/0.02_H); no longer U1.2 (A4/0.03_H)
- net switch02: now also U1.2 (A4/0.03_H); no longer U1.3 (A10/0.28)
- net switch03: now also U1.3 (A10/0.28); no longer U1.4 (A11/0.29)
- net switch04: now also U1.4 (A11/0.29); no longer U1.5 (A8_SDA/0.04_H)
- net switch05: now also U1.5 (A8_SDA/0.04_H); no longer U1.6 (A9_SCL/0.05_H)
- net switch06: now also U1.11 (A6_MOSI/1.15); no longer U1.7 (B8_TX/1.11)
- net switch07: now also U1.10 (A5_MISO/1.14); no longer U1.8 (B9_RX/1.12)
- net switch09: now also U1.8 (B9_RX/1.12); no longer U1.10 (A5_MISO/1.14)
- net switch10: now also U1.7 (B8_TX/1.11); no longer U1.11 (A6_MOSI/1.15)
- net at M1.2 (-), Q1.1 (C): now also D2.2 (A)
- net +3.3V: now reaches U1.12 (3V3)
- net +3.3V: now also M1.1 (+), D2.1 (K)
- net +5V: no longer names the net of U1.14 (5V)
- net +5V: no longer M1.1 (+)
